Commit message: modified:   epson_c3_support/urdf/c3_macro.xacro

File: epson_c3_support/urdf/c3_macro.xacro (robot description, xacro)
@@ -160,5 +160,5 @@
     </joint>
     <joint name="${prefix}joint_6" type="revolute">
-      <origin xyz="0 0.06 0" rpy="-1.570796326 -1.570796326 0"/>
+      <origin xyz="0 0.06 0" rpy="0 0 0"/>
       <parent link="${prefix}link_5"/>
       <child link="${prefix}link_6"/>
@@ -167,5 +167,5 @@
     </joint>
     <joint name="${prefix}joint_6-tool0" type="fixed">
-      <origin xyz="0 0 0.005" rpy="0 0 0.785398163" />
+      <origin xyz="0 0.005 0" rpy="-1.570796326 -1.570796326 0" />
       <parent link="${prefix}link_6"/>
       <child link="${prefix}tool0"/>

Commit message: modified:   epson_c3_support/urdf/c3_macro.xacro

File: epson_c3_support/urdf/c3_macro.xacro (robot description, xacro)
@@ -107,5 +107,5 @@
     <link name="${prefix}link_6">
       <visual>
-        <origin xyz="-0.57 0 -0.41" rpy="1.570796326 0 1.570796326"/>
+        <origin xyz="0 -0.41 -0.57" rpy="0 0 0"/>
         <geometry>
           <mesh filename="package://epson_c3_support/meshes/c3/visual/link_6.stl" scale="0.001 0.001 0.001" />
@@ -116,5 +116,5 @@
       </visual>
       <collision>
-        <origin xyz="-0.57 0 -0.41" rpy="1.570796326 0 1.570796326"/>
+        <origin xyz="0 -0.41 -0.57" rpy="0 0 0"/>
         <geometry>
           <mesh filename="package://epson_c3_support/meshes/c3/collision/link_6.stl" scale="0.001 0.001 0.001" />
@@ -163,5 +163,5 @@
       <parent link="${prefix}link_5"/>
       <child link="${prefix}link_6"/>
-      <axis xyz="0 0 -1"/>
+      <axis xyz="0 -1 0"/>
       <limit lower="-6.2832" upper="6.2832" effort="0" velocity="12.56"/>
     </joint>

Commit message: modified:   epson_c3_support/urdf/c3_macro.xacro

File: epson_c3_support/urdf/c3_macro.xacro (robot description, xacro)
@@ -167,5 +167,5 @@
     </joint>
     <joint name="${prefix}joint_6-tool0" type="fixed">
-      <origin xyz="0 0.005 0" rpy="-1.570796326 -1.570796326 0" />
+      <origin xyz="0 0.005 0" rpy="-1.047197551 -1.570796327 -0.523598776" />
       <parent link="${prefix}link_6"/>
       <child link="${prefix}tool0"/>

Commit message: modified:   epson_c3_support/urdf/c3_macro.xacro

File: epson_c3_support/urdf/c3_macro.xacro (robot description, xacro)
@@ -167,5 +167,5 @@
     </joint>
     <joint name="${prefix}joint_6-tool0" type="fixed">
-      <origin xyz="0 0.005 0" rpy="-1.047197551 -1.570796327 -0.523598776" />
+      <origin xyz="0 0.005 0" rpy="-1.570796327 -1.570796327 0" />
       <parent link="${prefix}link_6"/>
       <child link="${prefix}tool0"/>
